File: src/Eagle/CANFD_HUB.sch (EAGLE design)
At the start: 25 parts

Commit message: [complete]CANFD_HUB
Parts:
- added H1, H2, H3, H4: MOUNT-HOLE3.2(NORESIST), MOUNT-HOLE3.2(NORESIST):MOUNT-HOLE3.2(NORESIST)
Connections:
- net CAN_H renamed CAN_H+
- net CAN_L renamed CAN_L-
- net GND: now also H1.P$1, H2.P$1, H3.P$1, H4.P$1
- net LED1: now also SV1.4; no longer SV1.10
- net LED2: now also SV1.6; no longer SV1.9
- net LED4: now also SV1.10; no longer SV1.7
- net LED5: now also SV1.9; no longer SV1.6
- net LED6: now also SV1.7; no longer SV1.5
- net LED7: now also SV1.5; no longer SV1.4
